File: Eagle_Files/Clock.brd (EAGLE design)
At the start: 42.7 x 18.9 mm, 24 parts, among them IC1 MEGA8-AI, IC2 DS3231/SO, X1 332-02

Commit message: Adding usb connector intead of DC jack
Parts:
- removed J1: (no value), con-jack:DCJ0303
- added CN1: (no value), adafruit:USB-MINIB
- moved LOGO2 6.38 mm to (31.9, 2.46)
- moved C3 0.41 mm to (34.8, 11.8)
- moved R7 0.32 mm to (34.8, 13.1)
- moved R8 0.30 mm to (34.8, 14.6)
Connections:
- net GND: now also CN1.GND; no longer J1.2, J1.3
- net VCC: now also CN1.VBUS; no longer J1.1
Routing:
- net VCC: track 86.1 -> 91.3 mm, vias 3 -> 4
- net 4G: track 31.8 -> 31.2 mm
- net GND: vias 14 -> 11
